File: system_design/V0.5/PCB Design/PCBINSITU.sch (KiCad schematic (older format))
At the start: 9 parts, among them U1 SD, U2 BATTERY, U3 SWITCH, U4 TURBIDITY, U5 PH, U6 TDS, U7 RTC, U8 74HC237

Commit message: Water Quality Sensor
Parts:
- U1: symbol New_Library:SD -> PCBINSITU-rescue:SD-New_Library
- U2: symbol New_Library:BATTERY -> PCBINSITU-rescue:BATTERY-New_Library
- U3: symbol New_Library:SWITCH -> PCBINSITU-rescue:SWITCH-New_Library
- U4: symbol New_Library:TURBIDITY -> PCBINSITU-rescue:TURBIDITY-New_Library
- U5: symbol New_Library:PH -> PCBINSITU-rescue:PH-New_Library
- U6: symbol New_Library:TDS -> PCBINSITU-rescue:TDS-New_Library
- U7: symbol New_Library:RTC -> PCBINSITU-rescue:RTC-New_Library
Changed lines of the file:
@@
 $EndComp
 $Comp
-L New_Library:SWITCH U3
+L PCBINSITU-rescue:SWITCH-New_Library U3
 U 1 1 6298FABC
 P 5550 2250
@@
 NoConn ~ 5450 2550
 $Comp
-L New_Library:BATTERY U2
+L PCBINSITU-rescue:BATTERY-New_Library U2
 U 1 1 629927B4
 P 5000 2500
@@
 	5550 2750 5100 2750
 $Comp
-L New_Library:PH U5
+L PCBINSITU-rescue:PH-New_Library U5
 U 1 1 62994B8A
 P 6950 3200
@@
 	6950 3750 7300 3750
 $Comp
-L New_Library:TDS U6
+L PCBINSITU-rescue:TDS-New_Library U6
 U 1 1 62998311
 P 7600 3200
@@
 $EndComp
 $Comp
-L New_Library:TURBIDITY U4
+L PCBINSITU-rescue:TURBIDITY-New_Library U4
 U 1 1 6299C203
 P 6900 4300
@@
 	7300 2650 7950 2650
 $Comp
-L New_Library:SD U1
+L PCBINSITU-rescue:SD-New_Library U1
 U 1 1 629A42A1
 P 4150 4900
@@
 	6150 2450 6150 2750
 $Comp
-L New_Library:RTC U7
+L PCBINSITU-rescue:RTC-New_Library U7
 U 1 1 629BB9D8
 P 8400 3550
