File: System_development/Jocassee/V0.5.0/PCB/V0.5.0/V0.5.0.kicad_sch (KiCad schematic)
At the start: 15 parts, among them U1 water_Battery, U2 SD, U3 switch, U4 Sensor, U5 Sensor, U6 DS3231M, U7 Sensor, U8 Temp

Commit message: V.05 BOM updated
Parts:
- C1: value C -> 0.1uF
- R1: value R -> 4.7K
- R2: value R -> 470
Changed lines of the file:
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@@
 		(dnp no)
 		(property "Reference" "A1"
-			(at 154.94 125.4506 0)
+			(at 146.05 123.19 0)
 			(effects
 				(font
@@
 		)
 		(property "Value" "Arduino_Nano_v3.x"
-			(at 154.94 127.762 0)
+			(at 155.448 130.556 0)
 			(effects
 				(font
@@
 		(dnp no)
 		(property "Reference" "U6"
-			(at 210.82 134.3406 0)
+			(at 209.296 122.174 0)
 			(effects
 				(font
@@
 		)
 		(property "Value" "DS3231M"
-			(at 210.82 136.652 0)
+			(at 200.914 132.334 0)
 			(effects
 				(font
@@
 			)
 		)
-		(property "Value" "R"
+		(property "Value" "4.7K"
 			(at 247.65 96.1136 90)
 			(effects
@@
 		(dnp no)
 		(property "Reference" "BT1"
-			(at 214.63 113.157 90)
+			(at 217.424 104.394 90)
 			(effects
 				(font
@@
 		)
 		(property "Value" "Battery_Cell"
-			(at 214.63 110.8456 90)
+			(at 218.948 110.236 90)
 			(effects
 				(font
@@
 		)
 		(property "Value" "GND"
-			(at 157.607 127.5842 0)
+			(at 159.512 127.762 0)
 			(effects
 				(font
@@
 		)
 		(property "Value" "GND"
-			(at 155.067 127.5842 0)
+			(at 153.416 127.508 0)
 			(effects
 				(font
@@
 			)
 		)
-		(property "Value" "C"
+		(property "Value" "0.1uF"
 			(at 129.921 51.943 0)
 			(effects
@@
 			)
 		)
-		(property "Value" "R"
+		(property "Value" "470"
 			(at 115.57 60.5536 90)
 			(effects
