File: System_development/Jocassee/V0.5.0/PCB/V0.5.0/V0.5.0.kicad_pcb (KiCad board)
At the start: 2 copper layers, 32.6 x 97.2 mm, 16 parts, among them U1 water_Battery, U2 SD, U3 switch, U4 Sensor, U5 Sensor, U6 DS3231M, U7 Sensor, U8 Temp

Commit message: V0.5.0 PCB Update
Other:
- board text added: "Matthew Burnett"
- board text added: "V0.5.0\"
- board text removed: "V0.1\"
Changed lines of the file:
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@@
 	)
 	(gr_text "Joud Satme"
-		(at 113.5 117.1 0)
+		(at 113.324878 118.39123 0)
+		(layer "F.SilkS")
+		(effects
+			(font
+				(size 0.9 0.9)
+				(thickness 0.2)
+			)
+		)
+	)
+	(gr_text "Matthew Burnett"
+		(at 113 114 0)
 		(layer "F.SilkS")
 		(effects
@@
 	)
 	(gr_text "In-Situ Water Quality Sensor"
-		(at 117.5 112.7 0)
+		(at 116.3 112.7 0)
 		(layer "F.SilkS")
 		(effects
@@
 		)
 	)
-	(gr_text "V0.1\\"
-		(at 105.2 112.6 0)
+	(gr_text "V0.5.0\\"
+		(at 103.721423 112.584747 0)
 		(layer "F.SilkS")
 		(effects
@@
 	)
 	(gr_text "Antonio Fonce"
-		(at 112.6 115.6 0)
+		(at 112.424878 116.89123 0)
 		(layer "F.SilkS")
 		(effects
@@
 	)
 	(gr_text "Mohamed Abdelwahab"
-		(at 113.9 114.2 0)
+		(at 113.724878 115.49123 0)
 		(layer "F.SilkS")
 		(effects

Commit message: V 0.5 PCB errors corrected
Parts:
- U4: value Sensor -> pH
Other:
- board text added: "+"
- board text added: "A"
- board text added: "D"
- board text added: "GND"
- board text added: "LED"
- board text added: "TDS"
- board text added: "Turbidity"
Changed lines of the file:
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@@
 			(at -10.5 6.8 0)
 			(layer "F.SilkS")
+			(hide yes)
 			(effects
 				(font
@@
 			(layer "F.SilkS")
 		)
-		(fp_text user "Gnd"
-			(at -11.5 5.56 0)
-			(layer "F.SilkS")
-			(effects
-				(font
-					(size 0.4 0.5)
-					(thickness 0.09)
-				)
-			)
-		)
-		(fp_text user "+"
-			(at -8.9 5.6 0)
-			(layer "F.SilkS")
-			(effects
-				(font
-					(size 0.4 0.4)
-					(thickness 0.075)
-				)
-			)
-		)
-		(fp_text user "A"
-			(at -6.4 5.6 0)
-			(layer "F.SilkS")
-			(effects
-				(font
-					(size 0.3 0.4)
-					(thickness 0.05)
-				)
-			)
-		)
 		(pad "1" thru_hole circle
 			(at -11.48 4.41)
@@
 			)
 		)
-		(property "Value" "Sensor"
-			(at -8.4 7 0)
+		(property "Value" "pH"
+			(at -8.8 8.3 0)
 			(layer "F.SilkS")
 			(effects
 				(font
-					(size 0.6 0.6)
+					(size 1 1)
 					(thickness 0.12)
 				)
@@
 		)
 		(fp_text user "Gnd"
-			(at -11.5 5.56 0)
+			(at -11.5 6.8 0)
 			(layer "F.SilkS")
 			(effects
 				(font
-					(size 0.4 0.5)
+					(size 0.7 0.7)
 					(thickness 0.09)
 				)
@@
 		)
 		(fp_text user "+"
-			(at -8.9 5.6 0)
+			(at -8.9 6.8 0)
 			(layer "F.SilkS")
 			(effects
 				(font
-					(size 0.4 0.4)
+					(size 0.7 0.7)
 					(thickness 0.08)
 				)
@@
 		)
 		(fp_text user "A"
-			(at -6.35 5.6 0)
+			(at -6.35 6.8 0)
 			(layer "F.SilkS")
 			(effects
 				(font
-					(size 0.4 0.4)
+					(size 0.7 0.7)
 					(thickness 0.075)
 				)
@@
 			(at -7.7 6.9 0)
 			(layer "F.SilkS")
+			(hide yes)
 			(effects
 				(font
@@
 		)
 		(fp_text user "Gnd"
-			(at -11.5 5.56 0)
+			(at -11.5 6.8 0)
 			(layer "F.SilkS")
 			(effects
 				(font
-					(size 0.4 0.5)
+					(size 0.7 0.7)
 					(thickness 0.09)
 				)
@@
 		)
 		(fp_text user "+"
-			(at -8.4 5.55 0)
+			(at -9.1 6.8 0)
 			(layer "F.SilkS")
 			(effects
 				(font
-					(size 0.4 0.5)
+					(size 0.7 0.7)
 					(thickness 0.08)
 				)
@@
 		)
 		(fp_text user "A"
-			(at -6.35 5.55 0)
+			(at -6.35 6.8 0)
 			(layer "F.SilkS")
 			(effects
 				(font
-					(size 0.4 0.5)
+					(size 0.7 0.7)
 					(thickness 0.08)
 				)
@@
 			(layer "F.SilkS")
 		)
-		(fp_text user "+"
-			(at -8.9 5.7 0)
-			(layer "F.SilkS")
-			(effects
-				(font
-					(size 0.4 0.5)
-					(thickness 0.08)
-				)
-			)
-		)
-		(fp_text user "Gnd"
-			(at -11.5 5.56 0)
-			(layer "F.SilkS")
-			(effects
-				(font
-					(size 0.4 0.5)
-					(thickness 0.09)
-				)
-			)
-		)
-		(fp_text user "D"
-			(at -6.4 5.7 0)
-			(layer "F.SilkS")
-			(effects
-				(font
-					(size 0.4 0.5)
-					(thickness 0.08)
-				)
-			)
-		)
 		(pad "1" thru_hole circle
 			(at -11.48 4.41)
@@
 			(at 1.27 2.96 180)
 			(layer "F.Fab")
-			(hide yes)
 			(effects
 				(font
@@
 		)
 	)
+	(gr_text "GND"
+		(at 110 123.5 0)
+		(layer "F.SilkS")
+		(effects
+			(font
+				(size 0.7 0.7)
+				(thickness 0.12)
+			)
+		)
+	)
+	(gr_text "GND"
+		(at 111 81 0)
+		(layer "F.SilkS")
+		(effects
+			(font
+				(size 0.7 0.7)
+				(thickness 0.12)
+			)
+		)
+	)
+	(gr_text "TDS"
+		(at 122.5 82.5 0)
+		(layer "F.SilkS")
+		(effects
+			(font
+				(size 1 1)
+				(thickness 0.12)
+			)
+		)
+	)
+	(gr_text "A"
+		(at 116 81 0)
+		(layer "F.SilkS")
+		(effects
+			(font
+				(size 0.7 0.7)
+				(thickness 0.12)
+			)
+		)
+	)
 	(gr_text "Joud Satme"
 		(at 113.324878 118.39123 0)
@@
 		)
 	)
+	(gr_text "Turbidity"
+		(at 113.5 82.5 0)
+		(layer "F.SilkS")
+		(effects
+			(font
+				(size 1 1)
+				(thickness 0.12)
+			)
+		)
+	)
+	(gr_text "LED"
+		(at 121 54 0)
+		(layer "F.SilkS")
+		(effects
+			(font
+				(size 0.7 0.7)
+				(thickness 0.12)
+			)
+		)
+	)
 	(gr_text "Matthew Burnett"
 		(at 113 114 0)
@@
 		)
 	)
+	(gr_text "+"
+		(at 113 123.5 0)
+		(layer "F.SilkS")
+		(effects
+			(font
+				(size 0.7 0.7)
+				(thickness 0.12)
+			)
+		)
+	)
 	(gr_text "Mohamed Abdelwahab"
 		(at 113.724878 115.49123 0)
@@
 			)
 		)
+	)
+	(gr_text "D"
+		(at 115.5 123.5 0)
+		(layer "F.SilkS")
+		(effects
+			(font
+				(size 0.7 0.7)
+				(thickness 0.12)
+			)
+		)
+	)
+	(gr_text "+"
+		(at 113.5 81 0)
+		(layer "F.SilkS")
+		(effects
+			(font
+				(size 0.7 0.7)
+				(thickness 0.14)
+				(bold yes)
+			)
+		)

Commit message: V0.5 BOM updated
Parts:
- moved G*** 2.97 mm to (111.0, 102.0)
Other:
- board text added: "Arduino Nano"
- board text added: "Micro SD card"
Changed lines of the file:
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@@
 			(outputformat 1)
 			(mirror no)
-			(drillshape 1)
+			(drillshape 0)
 			(scaleselection 1)
-			(outputdirectory "")
+			(outputdirectory "Gerber Files/")
 		)
 	)
@@
 		)
 		(property "Value" "Temp"
-			(at -9.1 2 0)
+			(at -14.3 4.5 -90)
 			(layer "F.SilkS")
 			(effects
@@
 	(footprint "WATER_SENSOR:uofsc_logo_1in"
 		(layer "F.Cu")
-		(at 113.5 103.6)
+		(at 111 102)
 		(property "Reference" "G***"
 			(at 0 0 0)
@@
 		(layer "Edge.Cuts")
 	)
+	(gr_text "Micro SD card"
+		(at 113.5 103.6 -0)
+		(layer "B.SilkS")
+		(effects
+			(font
+				(size 1.2 1.2)
+				(thickness 0.2)
+				(bold yes)
+			)
+			(justify mirror)
+		)
+	)
 	(gr_text "#"
 		(at 116.9 36.5 180)
@@
 	)
 	(gr_text "Joud Satme"
-		(at 113.324878 118.39123 0)
+		(at 110.924878 116.99123 0)
 		(layer "F.SilkS")
 		(effects
@@
 		)
 	)
+	(gr_text "Arduino Nano"
+		(at 106.99 53.55 90)
+		(layer "F.SilkS")
+		(effects
+			(font
+				(size 1.2 1.2)
+				(thickness 0.2)
+				(bold yes)
+			)
+		)
+	)
 	(gr_text "Turbidity"
 		(at 113.5 82.5 0)
@@
 	)
 	(gr_text "Matthew Burnett"
-		(at 113 114 0)
+		(at 110.6 112.6 0)
 		(layer "F.SilkS")
 		(effects
@@
 	)
 	(gr_text "In-Situ Water Quality Sensor"
-		(at 116.3 112.7 0)
+		(at 113.9 111.3 0)
 		(layer "F.SilkS")
 		(effects
@@
 	)
 	(gr_text "V0.5.0\\"
-		(at 103.721423 112.584747 0)
+		(at 101.321423 111.184747 0)
 		(layer "F.SilkS")
 		(effects
@@
 	)
 	(gr_text "Antonio Fonce"
-		(at 112.424878 116.89123 0)
+		(at 110.024878 115.49123 0)
 		(layer "F.SilkS")
 		(effects
@@
 	)
 	(gr_text "Mohamed Abdelwahab"
-		(at 113.724878 115.49123 0)
+		(at 111.324878 114.09123 0)
 		(layer "F.SilkS")
 		(effects
@@
 	)
 	(gr_text "Arts Lab"
-		(at 112.4 110.9 0)
+		(at 110 109.5 0)
 		(layer "F.SilkS")
 		(effects

Commit message: V0.5 PCB refined
Routing:
- net GND: track 8.95 -> 0.00 mm, vias 22 -> 21
Other:
- outline, holes or cut-outs redrawn
- board text added: "Coin cell"
- board text added: "DS3231"
Changed lines of the file:
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@@
 	)
 	(gr_circle
-		(center 101.5 87.85)
-		(end 101.5 86.35)
+		(center 101.5 86.5)
+		(end 101.5 85)
 		(stroke
 			(width 0.05)
@@
 	)
 	(gr_circle
-		(center 125.5 87.85)
-		(end 125.5 86.35)
+		(center 125.5 86.5)
+		(end 125.5 85)
 		(stroke
 			(width 0.05)
@@
 		(layer "Edge.Cuts")
 	)
+	(gr_text "Coin cell"
+		(at 128.5 65 90)
+		(layer "B.SilkS")
+		(effects
+			(font
+				(size 1.2 1.2)
+				(thickness 0.2)
+				(bold yes)
+			)
+			(justify mirror)
+		)
+	)
+	(gr_text "DS3231"
+		(at 123 41 -0)
+		(layer "B.SilkS")
+		(effects
+			(font
+				(size 1.2 1.2)
+				(thickness 0.2)
+				(bold yes)
+			)
+			(justify mirror)
+		)
+	)
 	(gr_text "Micro SD card"
 		(at 113.5 103.6 -0)
@@
 		(net 5)
 	)
-	(segment
-		(start 125.75 104)
-		(end 127.158103 102.591897)
-		(width 0.25)
-		(layer "F.Cu")
+	(via
+		(at 101.5 34.5)
+		(size 0.8)
+		(drill 0.4)
+		(layers "F.Cu" "B.Cu")
 		(net 6)
 	)
-	(segment
-		(start 127.158103 97.558103)
-		(end 125.8 96.2)
-		(width 0.25)
-		(layer "F.Cu")
+	(via
+		(at 106.6 31.8)
+		(size 0.8)
+		(drill 0.4)
+		(layers "F.Cu" "B.Cu")
 		(net 6)
 	)
-	(segment
-		(start 127.158103 102.591897)
-		(end 127.158103 97.558103)
-		(width 0.25)
-		(layer "F.Cu")
+	(via
+		(at 114 28.8)
+		(size 0.8)
+		(drill 0.4)
+		(layers "F.Cu" "B.Cu")
 		(net 6)
 	)
 	(via
-		(at 101.5 34.5)
+		(at 126.5 57.4)
 		(size 0.8)
 		(drill 0.4)
@@
 	)
 	(via
-		(at 106.6 31.8)
+		(at 120.7 121.9)
 		(size 0.8)
 		(drill 0.4)
@@
 	)
 	(via
-		(at 114 28.8)
+		(at 101.7 29)
 		(size 0.8)
 		(drill 0.4)
@@
 	)
 	(via
-		(at 126.5 57.4)
-		(size 0.8)
-		(drill 0.4)
-		(layers "F.Cu" "B.Cu")
-		(net 6)
-	)
-	(via
-		(at 120.7 121.9)
-		(size 0.8)
-		(drill 0.4)
-		(layers "F.Cu" "B.Cu")
-		(net 6)
-	)
-	(via
-		(at 101.7 29)
-		(size 0.8)
-		(drill 0.4)
-		(layers "F.Cu" "B.Cu")
-		(net 6)
-	)
-	(via
 		(at 123.3 119.5)
 		(size 0.8)
 		(drill 0.4)
-		(layers "F.Cu" "B.Cu")
-		(net 6)
-	)
-	(via
-		(at 125.8 96.2)
-		(size 0.8)
-		(drill 0.4)
